Commit message: Updated packages

File: buraqbot_ws/src/buraq_description/urdf/buraq_ros2_control.urdf.xacro (robot description, xacro)
@@ -1,55 +1,67 @@
 <?xml version="1.0"?>
 <robot xmlns:xacro="http://www.ros.org/wiki/xacro">
-  <xacro:macro name="buraq_ros2_control" params="name prefix">
+  <xacro:macro name="buraq_ros2_control" params="name">
     <ros2_control name="${name}" type="system">
       <hardware>
         <plugin>buraq_hw/DiffDriveBuraq</plugin>
         <!-- Wheel joint names -->
-        <param name="front_left_wheel_name">${prefix}front_left_wheel_joint</param>
-        <param name="front_right_wheel_name">${prefix}front_right_wheel_joint</param>
-        <param name="rear_left_wheel_name">${prefix}rear_left_wheel_joint</param>
-        <param name="rear_right_wheel_name">${prefix}rear_right_wheel_joint</param>
+        <param name="front_left_wheel_name">front_left_wheel_joint</param>
+        <param name="front_right_wheel_name">front_right_wheel_joint</param>
+        <param name="rear_left_wheel_name">rear_left_wheel_joint</param>
+        <param name="rear_right_wheel_name">rear_right_wheel_joint</param>
         <!-- Serial communication parameters -->
         <param name="serial_device">/dev/ttyACM0</param>
-        <param name="baud_rate">115200</param>
+        <param name="baud_rate">57600</param>
         <param name="timeout">1000</param>
         <!-- Hardware parameters -->
         <param name="loop_rate">30</param>
-        <param name="front_left_enc_counts_per_rev">2410</param>
-        <param name="front_right_enc_counts_per_rev">2452</param>
-        <param name="rear_left_enc_counts_per_rev">2369</param>
-        <param name="rear_right_enc_counts_per_rev">2327</param>
+        <param name="front_left_enc_counts_per_rev">2390</param>
+        <param name="front_right_enc_counts_per_rev">2390</param>
+        <param name="rear_left_enc_counts_per_rev">2390</param>
+        <param name="rear_right_enc_counts_per_rev">2390</param>
         <!-- PID parameters -->
-        <param name="pid_p">0.3</param>
-        <param name="pid_i">0.05</param>
-        <param name="pid_d">0.005</param>
-        <param name="pid_o">0.8</param>
+        <param name="pid_p">0.2</param>
+        <param name="pid_i">0.001</param>
+        <param name="pid_d">0.0</param>
+        <param name="pid_o">1.0</param>
       </hardware>
       <!-- Front Left Wheel -->
-      <joint name="${prefix}front_left_wheel_joint">
-        <command_interface name="velocity"/>
+      <joint name="front_left_wheel_joint">
+        <command_interface name="velocity">
+          <param name="min">-5</param>
+          <param name="max">5</param>
+        </command_interface>
         <state_interface name="position"/>
         <state_interface name="velocity"/>
       </joint>
       <!-- Front Right Wheel -->
-      <joint name="${prefix}front_right_wheel_joint">
-        <command_interface name="velocity"/>
+      <joint name="front_right_wheel_joint">
+        <command_interface name="velocity">
+          <param name="min">-5</param>
+          <param name="max">5</param>
+        </command_interface>
         <state_interface name="position"/>
         <state_interface name="velocity"/>
       </joint>
       <!-- Rear Left Wheel -->
-      <joint name="${prefix}rear_left_wheel_joint">
-        <command_interface name="velocity"/>
+      <joint name="rear_left_wheel_joint">
+        <command_interface name="velocity">
+          <param name="min">-5</param>
+          <param name="max">5</param>
+        </command_interface>
         <state_interface name="position"/>
         <state_interface name="velocity"/>
       </joint>
       <!-- Rear Right Wheel -->
-      <joint name="${prefix}rear_right_wheel_joint">
-        <command_interface name="velocity"/>
+      <joint name="rear_right_wheel_joint">
+        <command_interface name="velocity">
+          <param name="min">-5</param>
+          <param name="max">5</param>
+        </command_interface>
         <state_interface name="position"/>
         <state_interface name="velocity"/>
       </joint>
       <!-- IMU Sensor -->
-      <sensor name="imu_sensor">
+      <sensor name="imu">
         <state_interface name="orientation.x"/>
         <state_interface name="orientation.y"/>
